File: hw/sch_pcb/I2CIO01.kicad_pcb (KiCad board)
At the start: 2 copper layers, 40.1 x 40.1 mm, 38 parts, among them J1 JUMP_2X2, J2 JUMP_5X2, J3 JUMP_3X2, J4 CONN_2, J5 CONN1_2, J6 JUMP_8X2, J7 JUMP_8X2, J8 CONN1_2, J9 CONN_2, P1 _, P2 _, P3 _, P4 _, U1 TCA6416A

Commit message: Update PCB to KiCADv7.
Other:
- net class Default removed
- net class vdd removed
